Commit message: feat(robot): update robot URDF and launch file for state publishing; modify lidar node for distance handling

File: src/my_robot_bringup/config/robot.urdf (robot description, URDF)
Before this commit: robot abc_robot, 4 links, 3 joints
Joints:
- joint camera_joint: origin xyz=0.1 0.0 0.08 rpy=0 0 0 -> xyz=0 0 0 rpy=0 0 0

Commit message: feat(robot.urdf): update joint origin positions for imu, laser, and camera links

File: src/my_robot_bringup/config/robot.urdf (robot description, URDF)
Before this commit: robot abc_robot, 4 links, 3 joints
Joints:
- joint camera_joint: origin xyz=0 0 0 rpy=0 0 0 -> xyz=0.0575 0 0.177 rpy=0 0 0
- joint imu_joint: origin xyz=0 0 0 rpy=0 0 0 -> xyz=0.012 -0.015 0.0805 rpy=0 0 0
- joint laser_joint: origin xyz=0 0 0 rpy=0 0 0 -> xyz=0 0 0.1461 rpy=0 0 0

Commit message: fix(robot.urdf): correct camera joint orientation in URDF configuration

File: src/my_robot_bringup/config/robot.urdf (robot description, URDF)
Before this commit: robot abc_robot, 4 links, 3 joints
Joints:
- joint camera_joint: origin xyz=0.0575 0 0.177 rpy=0 0 0 -> xyz=0.0575 0 0.177 rpy=3.1415926 0 0

Commit message: feat: add VINS-Fusion configuration files and update image splitter rotation angle

File: src/my_robot_bringup/config/robot.urdf (robot description, URDF)
Before this commit: robot abc_robot, 4 links, 3 joints
Joints:
- joint camera_joint: origin xyz=0.0575 0 0.177 rpy=3.1415926 0 0 -> xyz=0.0575 0 0.177 rpy=0 0 0

Commit message: feat: add CycloneDDS configuration for remote RVIZ2 access and update image splitter parameters

File: src/my_robot_bringup/config/robot.urdf (robot description, URDF)
Before this commit: robot abc_robot, 4 links, 3 joints
Links:
- added link left_camera_link
- added link right_camera_link
Joints:
- added joint left_camera_joint: type fixed, parent camera_link, child left_camera_link, origin xyz=0 0.02875 0 rpy=0 0 0
- added joint right_camera_joint: type fixed, parent camera_link, child right_camera_link, origin xyz=0 -0.02875 0 rpy=0 0 0

Commit message: feat(vslam): adapt image splitter for Isaac ROS cuVSLAM and add dedicated launch
- Add mono8 encoding support and decouple compressed publish FPS in image_splitter_node
- Inject calibrated camera intrinsics, distortion coefficients, and exact baseline (51.912mm) into CameraInfo
- Add left/right camera optical frames with standard ROS optical rotation in robot.urdf
- Disable auto_log by default in params.yaml and robot.launch.py
- Add isaac_visual_slam.launch.py supporting ground constraint and simulation clock
- Add isaac_visual_slam.rviz with preconfigured odometry, path, and feature point clouds
- Update README.md and submodule references

File: src/my_robot_bringup/config/robot.urdf (robot description, URDF)
Before this commit: robot abc_robot, 6 links, 5 joints
Links:
- added link left_camera_optical_frame
- added link right_camera_optical_frame
Joints:
- added joint left_camera_optical_joint: type fixed, parent left_camera_link, child left_camera_optical_frame, origin xyz=0 0 0 rpy=-1.57079632679 0 -1.57079632679
- added joint right_camera_optical_joint: type fixed, parent right_camera_link, child right_camera_optical_frame, origin xyz=0 0 0 rpy=-1.57079632679 0 -1.57079632679
- joint left_camera_joint: origin xyz=0 0.02875 0 rpy=0 0 0 -> xyz=0 0.025956 0 rpy=0 0 0
- joint right_camera_joint: origin xyz=0 -0.02875 0 rpy=0 0 0 -> xyz=0 -0.025956 0 rpy=0 0 0

Commit message: feat(perception): upgrade stereo camera node with hardware acceleration, multi-rate streaming, and optical TF
- Refactor image_splitter_node as a ROS 2 Composable Node (ImageSplitterNode) for zero-copy IPC support.
- Implement GStreamer pipeline with SIMD JPEG decoding and Jetson VIC (nvvidconv) hardware 180° rotation (72+ FPS).
- Support multi-rate streaming: BGR8 stream at 15 Hz for AI detection, Mono8 stream at 60 Hz with 3x3 Gaussian filtering for cuVSLAM/VIO, and Compressed JPEG stream at 15 Hz.
- Add GStreamer plugin isolation sandbox (setup_clean_gstreamer_environment) to prevent CSI Argus daemon socket probe and GLib abort on USB cameras.
- Fix cv_bridge sub-matrix serialization bus error (SIGBUS) by ensuring continuous ROI memory layout with .clone().
- Add sensor Auto-Exposure/Auto-White-Balance warmup frames upon camera initialization.
- Add left_camera_optical_frame and right_camera_optical_frame to robot.urdf (REP-103 standard) for seamless RViz2 and VSLAM projection.
- Update Dockerfile with gstreamer1.0-plugins-good and gstreamer1.0-tools.
- Update data_logger_node to record stereo mono topics.
- Update perception package documentation in README.md.

File: src/my_robot_bringup/config/robot.urdf (robot description, URDF)
Before this commit: robot abc_robot, 6 links, 5 joints
Links:
- added link left_camera_optical_frame
- added link right_camera_optical_frame
Joints:
- added joint left_camera_optical_joint: type fixed, parent left_camera_link, child left_camera_optical_frame, origin xyz=0 0 0 rpy=-1.5707963267948966 0 -1.5707963267948966
- added joint right_camera_optical_joint: type fixed, parent right_camera_link, child right_camera_optical_frame, origin xyz=0 0 0 rpy=-1.5707963267948966 0 -1.5707963267948966

Commit message: feat(perception): implement hardware timestamp compensation and update calibration parameters
- Add timestamp_offset_ms parameter to image_splitter_node with automatic 33ms hardware exposure rollback compensation.
- Optimize image_splitter_node with static pre-allocated CameraInfo buffers for zero-allocation publishing.
- Update GStreamer capture pipeline with zero-buffering (appsink max-buffers=1 drop=1 sync=false) and v4l2src do-timestamp=true.
- Update stereo camera baseline in robot.urdf to calibrated 51.912mm (y = ±0.025956m).
- Synchronize vins_fusion_stereo_imu_config.yaml with latest Kalibr calibration extrinsics, switch topics to 60 Hz mono streams, and reset td to 0.0.
- Save latest Kalibr calibration results in src/my_robot_perception/doc/Calibration/.
- Update vi_car calibration configuration in src/vins_fusion submodule.

File: src/my_robot_bringup/config/robot.urdf (robot description, URDF)
Before this commit: robot abc_robot, 8 links, 7 joints
Joints:
- joint left_camera_joint: origin xyz=0 0.02875 0 rpy=0 0 0 -> xyz=0 0.025956 0 rpy=0 0 0
- joint right_camera_joint: origin xyz=0 -0.02875 0 rpy=0 0 0 -> xyz=0 -0.025956 0 rpy=0 0 0
